Commit message: feat(bringup): add simulation package for Gazebo Ignition
- Add launch files to spawn robot
- Verify basic simulation functionality

File: src/biped_description/urdf/biped.urdf.xacro (robot description, xacro)
@@ -3,5 +3,5 @@
   name="bipedal_robot">
   <!-- Define mesh directory variable -->
-  <xacro:property name="mesh_dir" value="package://biped_description/meshes"/>
+  <xacro:property name="mesh_dir" value="model://biped_description/meshes"/>
   <link
     name="base_link">
