Commit message: refactor(description, bringup, control) - bringup: add the gazebo resource path for the description package - description: rename biped.urdf.xacro to .urdf - control: minor correction

File: src/biped_description/urdf/biped.urdf (robot description, URDF)
Before this commit: robot bipedal_robot, 7 links, 6 joints
Links:
- added link imu_link, mass 0.001; visual box size=0.04 0.04 0.01
Joints:
- added joint imu_joint: type fixed, parent base_link, child imu_link, origin xyz=0.0 0.0 0.05 rpy=0.0 0.0 0.0

File: src/biped_description/urdf/biped_with_control.urdf.xacro (robot description, xacro)
@@ -5,4 +5,4 @@
     <xacro:include filename="$(find biped_description)/urdf/biped_sim_ros2_control.urdf" />
     <!-- robot description -->
-    <xacro:include filename="$(find biped_description)/urdf/biped.urdf.xacro" />
+    <xacro:include filename="$(find biped_description)/urdf/biped.urdf" />
 </robot>

Commit message: chore(description): add a new urdf.xacro beside the urdf file

File: src/biped_description/urdf/biped.urdf (robot description, URDF)
Before this commit: robot bipedal_robot, 8 links, 7 joints
Links:
- link base_link: geometry collision mesh filename=package://biped_description/meshes/base_link.STL; visual mesh filename=package://biped_description/meshes/base_link.STL
- link left_hip_pitch_link: geometry collision mesh filename=package://biped_description/meshes/left_hip_pitch_link.STL; visual mesh filename=package://biped_description/meshes/left_hip_pitch_link.STL
- link left_hip_roll_link: geometry collision mesh filename=package://biped_description/meshes/left_hip_roll_link.STL; visual mesh filename=package://biped_description/meshes/left_hip_roll_link.STL
- link left_knee_link: geometry collision mesh filename=package://biped_description/meshes/left_knee_link.STL; visual mesh filename=package://biped_description/meshes/left_knee_link.STL
- link right_hip_pitch_link: geometry collision mesh filename=package://biped_description/meshes/right_hip_pitch_link.STL; visual mesh filename=package://biped_description/meshes/right_hip_pitch_link.STL
- link right_hip_roll_link: geometry collision mesh filename=package://biped_description/meshes/right_hip_roll_link.STL; visual mesh filename=package://biped_description/meshes/right_hip_roll_link.STL
- link right_knee_link: geometry collision mesh filename=package://biped_description/meshes/right_knee_link.STL; visual mesh filename=package://biped_description/meshes/right_knee_link.STL

File: src/biped_description/urdf/biped_with_control.urdf.xacro (robot description, xacro)
@@ -5,4 +5,4 @@
     <xacro:include filename="$(find biped_description)/urdf/biped_sim_ros2_control.urdf" />
     <!-- robot description -->
-    <xacro:include filename="$(find biped_description)/urdf/biped.urdf" />
+    <xacro:include filename="$(find biped_description)/urdf/biped.urdf.xacro" />
 </robot>
